Commit message: sync https://www.lejuhub.com/highlydynamic/kuavo-ros-control/commit/359cbe56dcfb873bd42c45dde10a2b01b9e5c5cd

File: src/kuavo_assets/models/biped_s30/urdf/biped_s30.urdf (robot description, URDF)
Before this commit: robot biped_s4, 28 links, 27 joints
Links:
- link base_link: geometry visual mesh filename=package://kuavo_assets/models/biped_s40/meshes/torso.STL
- link leg_l1_link: geometry visual mesh filename=package://kuavo_assets/models/biped_s40/meshes/l_leg_roll.S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
- link leg_l2_link: geometry visual mesh filename=package://kuavo_assets/models/biped_s40/meshes/l_leg_yaw.STL
- link leg_l4_link: geometry visual mesh filename=package://kuavo_assets/models/biped_s40/meshes/l_knee.STL
- link leg_r1_link: geometry visual mesh filename=package://kuavo_assets/models/biped_s40/meshes/r_leg_roll.S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
- link leg_r2_link: geometry visual mesh filename=package://kuavo_assets/models/biped_s40/meshes/r_leg_yaw.STL
- link leg_r4_link: geometry visual mesh filename=package://kuavo_assets/models/biped_s40/meshes/r_knee.STL

File: src/kuavo_assets/models/biped_s30/urdf/drake/Lleg.urdf (robot description, URDF)
Before this commit: robot Lleg, 7 links, 4 joints
Links:
- link base_link: geometry visual mesh filename=../../meshes/l_knee.STL
- link l_foot_pitch: geometry visual mesh filename=../../meshes/l_foot_pitch.STL
- link l_foot_roll: geometry collision sphere radius=0.005; collision sphere radius=0.005
- link l_l_bar_y: geometry visual mesh filename=../../meshes/l_l_bar.STL
- link l_l_tendon_y: geometry visual mesh filename=../../meshes/l_l_tendon.STL
- link l_r_bar_y: geometry visual mesh filename=../../meshes/l_r_bar.STL
- link l_r_tendon_y: geometry visual mesh filename=../../meshes/l_r_tendon.STL

File: src/kuavo_assets/models/biped_s30/urdf/drake/Rleg.urdf (robot description, URDF)
Before this commit: robot Rleg, 7 links, 4 joints
Links:
- link base_link: geometry visual mesh filename=../../meshes/r_knee.STL
- link r_foot_pitch: geometry visual mesh filename=../../meshes/r_foot_pitch.STL
- link r_foot_roll: geometry collision sphere radius=0.005; collision sphere radius=0.005
- link r_l_bar_y: geometry visual mesh filename=../../meshes/r_l_bar.STL
- link r_l_tendon_y: geometry visual mesh filename=../../meshes/r_l_tendon.STL
- link r_r_bar_y: geometry visual mesh filename=../../meshes/r_r_bar.STL
- link r_r_tendon_y: geometry visual mesh filename=../../meshes/r_r_tendon.STL

File: src/kuavo_assets/models/biped_s30/urdf/drake/biped_v3.urdf (robot description, URDF)
Before this commit: robot biped_v3, 13 links, 12 joints
Links:
- link l_foot_pitch: geometry visual mesh filename=../../meshes/l_foot_pitch.STL
- link l_foot_roll: geometry collision sphere radius=0.005; collision sphere radius=0.005
- link l_knee: geometry visual mesh filename=../../meshes/l_knee.STL
- link l_leg_pitch: geometry visual mesh filename=../../meshes/l_leg_pitch.STL
- link l_leg_roll: geometry visual mesh filename=../../meshes/l_leg_roll.STL
- link l_leg_yaw: geometry visual mesh filename=../../meshes/l_leg_yaw.STL
- link r_foot_pitch: geometry visual mesh filename=../../meshes/r_foot_pitch.STL
- link r_foot_roll: geometry collision sphere radius=0.005; collision sphere radius=0.005
- link r_knee: geometry visual mesh filename=../../meshes/r_knee.STL
- link r_leg_pitch: geometry visual mesh filename=../../meshes/r_leg_pitch.STL
- link r_leg_roll: geometry visual mesh filename=../../meshes/r_leg_roll.STL
- link r_leg_yaw: geometry visual mesh filename=../../meshes/r_leg_yaw.STL
- link torso: geometry visual mesh filename=../../meshes/torso.STL

File: src/kuavo_assets/models/biped_s30/urdf/drake/biped_v3_all_joint.urdf (robot description, URDF)
Before this commit: robot biped_v3_all_joint, 35 links, 30 joints
Links:
- link l_foot_pitch: geometry visual mesh filename=../../meshes/l_foot_pitch.STL
- link l_foot_roll: geometry collision sphere radius=0.005; collision sphere radius=0.005
- link l_knee: geometry visual mesh filename=../../meshes/l_knee.STL
- link l_l_bar_y: geometry visual mesh filename=../../meshes/l_l_bar.STL
- link l_l_tendon_y: geometry visual mesh filename=../../meshes/l_l_tendon.STL
- link l_leg_pitch: geometry visual mesh filename=../../meshes/l_leg_pitch.STL
- link l_leg_roll: geometry visual mesh filename=../../meshes/l_leg_roll.STL
- link l_leg_yaw: geometry visual mesh filename=../../meshes/l_leg_yaw.STL
- link l_r_bar_y: geometry visual mesh filename=../../meshes/l_r_bar.STL
- link l_r_tendon_y: geometry visual mesh filename=../../meshes/l_r_tendon.STL
- link r_foot_pitch: geometry visual mesh filename=../../meshes/r_foot_pitch.STL
- link r_foot_roll: geometry collision sphere radius=0.005; collision sphere radius=0.005
- link r_knee: geometry visual mesh filename=../../meshes/r_knee.STL
- link r_l_bar_y: geometry visual mesh filename=../../meshes/r_l_bar.STL
- link r_l_tendon_y: geometry visual mesh filename=../../meshes/r_l_tendon.STL
- link r_leg_pitch: geometry visual mesh filename=../../meshes/r_leg_pitch.STL
- link r_leg_roll: geometry visual mesh filename=../../meshes/r_leg_roll.STL
- link r_leg_yaw: geometry visual mesh filename=../../meshes/r_leg_yaw.STL
- link r_r_bar_y: geometry visual mesh filename=../../meshes/r_r_bar.STL
- link r_r_tendon_y: geometry visual mesh filename=../../meshes/r_r_tendon.STL
- link torso: geometry visual mesh filename=../../meshes/torso.STL

File: src/kuavo_assets/models/biped_s30/urdf/drake/biped_v3_arm.urdf (robot description, URDF)
Before this commit: robot biped_v3_arm, 15 links, 14 joints
Links:
- link torso: geometry visual mesh filename=../../meshes/torso.STL

File: src/kuavo_assets/models/biped_s30/urdf/drake/biped_v3_full.urdf (robot description, URDF)
Before this commit: robot biped_v3_full, 27 links, 26 joints
Links:
- link l_foot_pitch: geometry visual mesh filename=../../meshes/l_foot_pitch.STL
- link l_foot_roll: geometry collision sphere radius=0.005; collision sphere radius=0.005
- link l_knee: geometry visual mesh filename=../../meshes/l_knee.STL
- link l_leg_pitch: geometry visual mesh filename=../../meshes/l_leg_pitch.STL
- link l_leg_roll: geometry visual mesh filename=../../meshes/l_leg_roll.STL
- link l_leg_yaw: geometry visual mesh filename=../../meshes/l_leg_yaw.STL
- link r_foot_pitch: geometry visual mesh filename=../../meshes/r_foot_pitch.STL
- link r_foot_roll: geometry collision sphere radius=0.005; collision sphere radius=0.005
- link r_knee: geometry visual mesh filename=../../meshes/r_knee.STL
- link r_leg_pitch: geometry visual mesh filename=../../meshes/r_leg_pitch.STL
- link r_leg_roll: geometry visual mesh filename=../../meshes/r_leg_roll.STL
- link r_leg_yaw: geometry visual mesh filename=../../meshes/r_leg_yaw.STL
- link torso: geometry visual mesh filename=../../meshes/torso.STL

File: src/kuavo_assets/models/biped_s31/urdf/biped_s31.urdf (robot description, URDF)
Before this commit: robot biped_s41, 28 links, 27 joints
Links:
- link base_link: geometry visual mesh filename=package://kuavo_assets/models/biped_s41/meshes/torso.STL

File: src/kuavo_assets/models/biped_s31/urdf/drake/biped_v3.urdf (robot description, URDF)
Before this commit: robot biped_v3, 13 links, 12 joints
Links:
- link torso: geometry visual mesh filename=../../meshes/torso.STL

File: src/kuavo_assets/models/biped_s31/urdf/drake/biped_v3_all_joint.urdf (robot description, URDF)
Before this commit: robot biped_v3_all_joint, 35 links, 30 joints
Links:
- link torso: geometry visual mesh filename=../../meshes/torso.STL

File: src/kuavo_assets/models/biped_s31/urdf/drake/biped_v3_arm.urdf (robot description, URDF)
Before this commit: robot biped_v3_arm, 15 links, 14 joints
Links:
- link torso: geometry visual mesh filename=../../meshes/torso.STL

File: src/kuavo_assets/models/biped_s31/urdf/drake/biped_v3_full.urdf (robot description, URDF)
Before this commit: robot biped_v3_full, 27 links, 26 joints
Links:
- link torso: geometry visual mesh filename=../../meshes/torso.STL

File: src/kuavo_assets/models/biped_s40/urdf/biped_s40.urdf (robot description, URDF)
Before this commit: robot biped_s4, 45 links, 44 joints
Links:
- link base_link: geometry visual mesh filename=package://kuavo_assets/models/biped_s40/meshes/torso.STL
- link leg_l1_link: geometry visual mesh filename=package://kuavo_assets/models/biped_s40/meshes/l_leg_roll.S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
- link leg_l2_link: geometry visual mesh filename=package://kuavo_assets/models/biped_s40/meshes/l_leg_yaw.STL
- link leg_l4_link: geometry visual mesh filename=package://kuavo_assets/models/biped_s40/meshes/l_knee.STL
- link leg_r1_link: geometry visual mesh filename=package://kuavo_assets/models/biped_s40/meshes/r_leg_roll.S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
- link leg_r2_link: geometry visual mesh filename=package://kuavo_assets/models/biped_s40/meshes/r_leg_yaw.STL
- link leg_r4_link: geometry visual mesh filename=package://kuavo_assets/models/biped_s40/meshes/r_knee.STL
- link zarm_l2_link: geometry visual mesh filename=package://kuavo_assets/models/biped_s40/meshes/l_arm_roll.S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
- link zarm_l3_link: geometry visual mesh filename=package://kuavo_assets/models/biped_s40/meshes/l_arm_yaw.STL
- link zarm_l5_link: geometry visual mesh filename=package://kuavo_assets/models/biped_s40/meshes/l_hand_yaw.S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
- link zarm_r2_link: geometry visual mesh filename=package://kuavo_assets/models/biped_s40/meshes/r_arm_roll.S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
- link zarm_r3_link: geometry visual mesh filename=package://kuavo_assets/models/biped_s40/meshes/r_arm_yaw.STL
- link zarm_r5_link: geometry visual mesh filename=package://kuavo_assets/models/biped_s40/meshes/r_hand_yaw.S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

File: src/kuavo_assets/models/biped_s40/urdf/drake/biped_v3.urdf (robot description, URDF)
Before this commit: robot biped_v3, 13 links, 12 joints
Links:
- link l_foot_pitch: geometry visual mesh filename=../../meshes/l_foot_pitch.STL
- link l_foot_roll: geometry collision sphere radius=0.005; collision sphere radius=0.005
- link l_knee: geometry visual mesh filename=../../meshes/l_knee.STL
- link l_leg_pitch: geometry visual mesh filename=../../meshes/l_leg_pitch.STL
- link l_leg_roll: geometry visual mesh filename=../../meshes/l_leg_roll.STL
- link l_leg_yaw: geometry visual mesh filename=../../meshes/l_leg_yaw.STL
- link r_foot_pitch: geometry visual mesh filename=../../meshes/r_foot_pitch.STL
- link r_foot_roll: geometry collision sphere radius=0.005; collision sphere radius=0.005
- link r_knee: geometry visual mesh filename=../../meshes/r_knee.STL
- link r_leg_pitch: geometry visual mesh filename=../../meshes/r_leg_pitch.STL
- link r_leg_roll: geometry visual mesh filename=../../meshes/r_leg_roll.STL
- link r_leg_yaw: geometry visual mesh filename=../../meshes/r_leg_yaw.STL
- link torso: geometry visual mesh filename=../../meshes/base_link.STL

File: src/kuavo_assets/models/biped_s40/urdf/drake/biped_v3_all_joint.urdf (robot description, URDF)
Before this commit: robot biped_v3_all_joint, 35 links, 30 joints
Links:
- link l_foot_pitch: geometry visual mesh filename=../../meshes/l_foot_pitch.STL
- link l_foot_roll: geometry collision sphere radius=0.005; collision sphere radius=0.005
- link l_knee: geometry visual mesh filename=../../meshes/l_knee.STL
- link l_l_bar_y: geometry visual mesh filename=../../meshes/l_l_bar.STL
- link l_l_tendon_y: geometry visual mesh filename=../../meshes/l_l_tendon.STL
- link l_leg_pitch: geometry visual mesh filename=../../meshes/l_leg_pitch.STL
- link l_leg_roll: geometry visual mesh filename=../../meshes/l_leg_roll.STL
- link l_leg_yaw: geometry visual mesh filename=../../meshes/l_leg_yaw.STL
- link l_r_bar_y: geometry visual mesh filename=../../meshes/l_r_bar.STL
- link l_r_tendon_y: geometry visual mesh filename=../../meshes/l_r_tendon.STL
- link r_foot_pitch: geometry visual mesh filename=../../meshes/r_foot_pitch.STL
- link r_foot_roll: geometry collision sphere radius=0.005; collision sphere radius=0.005
- link r_knee: geometry visual mesh filename=../../meshes/r_knee.STL
- link r_l_bar_y: geometry visual mesh filename=../../meshes/r_l_bar.STL
- link r_l_tendon_y: geometry visual mesh filename=../../meshes/r_l_tendon.STL
- link r_leg_pitch: geometry visual mesh filename=../../meshes/r_leg_pitch.STL
- link r_leg_roll: geometry visual mesh filename=../../meshes/r_leg_roll.STL
- link r_leg_yaw: geometry visual mesh filename=../../meshes/r_leg_yaw.STL
- link r_r_bar_y: geometry visual mesh filename=../../meshes/r_r_bar.STL
- link r_r_tendon_y: geometry visual mesh filename=../../meshes/r_r_tendon.STL
- link torso: geometry visual mesh filename=../../meshes/base_link.STL

File: src/kuavo_assets/models/biped_s40/urdf/drake/biped_v3_arm.urdf (robot description, URDF)
Before this commit: robot biped_v3_arm, 15 links, 14 joints
Links:
- link torso: geometry visual mesh filename=../../meshes/base_link.STL

File: src/kuavo_assets/models/biped_s40/urdf/drake/biped_v3_full.urdf (robot description, URDF)
Before this commit: robot biped_v3_full, 27 links, 26 joints
Links:
- link l_foot_pitch: geometry visual mesh filename=../../meshes/l_foot_pitch.STL
- link l_foot_roll: geometry collision sphere radius=0.005; collision sphere radius=0.005
- link l_knee: geometry visual mesh filename=../../meshes/l_knee.STL
- link l_leg_pitch: geometry visual mesh filename=../../meshes/l_leg_pitch.STL
- link l_leg_roll: geometry visual mesh filename=../../meshes/l_leg_roll.STL
- link l_leg_yaw: geometry visual mesh filename=../../meshes/l_leg_yaw.STL
- link r_foot_pitch: geometry visual mesh filename=../../meshes/r_foot_pitch.STL
- link r_foot_roll: geometry collision sphere radius=0.005; collision sphere radius=0.005
- link r_knee: geometry visual mesh filename=../../meshes/r_knee.STL
- link r_leg_pitch: geometry visual mesh filename=../../meshes/r_leg_pitch.STL
- link r_leg_roll: geometry visual mesh filename=../../meshes/r_leg_roll.STL
- link r_leg_yaw: geometry visual mesh filename=../../meshes/r_leg_yaw.STL
- link torso: geometry visual mesh filename=../../meshes/base_link.STL

File: src/kuavo_assets/models/biped_s41/urdf/biped_s41.urdf (robot description, URDF)
Before this commit: robot biped_s41, 45 links, 44 joints
Links:
- link base_link: geometry visual mesh filename=package://kuavo_assets/models/biped_s41/meshes/torso.STL

File: src/kuavo_assets/models/biped_s41/urdf/drake/biped_v3.urdf (robot description, URDF)
Before this commit: robot biped_v3, 13 links, 12 joints
Links:
- link torso: geometry visual mesh filename=../../meshes/base_link.STL

File: src/kuavo_assets/models/biped_s41/urdf/drake/biped_v3_all_joint.urdf (robot description, URDF)
Before this commit: robot biped_v3_all_joint, 35 links, 30 joints
Links:
- link torso: geometry visual mesh filename=../../meshes/base_link.STL
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