Commit message: sync https://www.lejuhub.com/highlydynamic/kuavo-ros-control/commit/fe176f4d1a57c70c1905d2560538ae831960852a

File: src/kuavo_assets/models/biped_s43/urdf/biped_s43.urdf (robot description, URDF)
Before this commit: robot biped_s4, 45 links, 44 joints
Joints:
- joint zarm_r2_joint: limit lower=-0.3489 upper=2.0933 effort=8.5 velocity=9 -> lower=0.3489 upper=-2.0933 effort=8.5 velocity=9
