Commit message: sync https://www.lejuhub.com/highlydynamic/kuavo-ros-control/commit/ee2295dc5ec7807fc888fd41c196baf72f387ad9

File: src/kuavo_assets/models/biped_s43/urdf/drake/biped_v3_arm.urdf (robot description, URDF)
Before this commit: robot biped_v3_arm, 17 links, 16 joints
Links:
- removed link zarm_l1_link
- removed link zarm_l2_link
- removed link zarm_l3_link
- removed link zarm_l4_link
- removed link zarm_l5_link
- removed link zarm_l6_link
- removed link zarm_l7_link
- removed link zarm_r1_link
- removed link zarm_r2_link
- removed link zarm_r3_link
- removed link zarm_r4_link
- removed link zarm_r5_link
- removed link zarm_r6_link
- removed link zarm_r7_link
- added link l_arm_pitch, mass 0.962; visual mesh filename=../../meshes/l_arm_pitch.STL
- added link l_arm_roll, mass 0.57; visual mesh filename=../../meshes/l_arm_roll.STL
- added link l_arm_yaw, mass 1.65; visual mesh filename=../../meshes/l_arm_yaw.STL
- added link l_forearm_pitch, mass 0.429; visual mesh filename=../../meshes/l_foream.STL
- added link l_hand_pitch, mass 0.331; visual mesh filename=../../meshes/l_hand_roll.STL
- added link l_hand_roll, mass 0.64; visual mesh filename=../../meshes/l_hand_pitch.STL
- added link l_hand_yaw, mass 0.61; visual mesh filename=../../meshes/l_hand_yaw.STL
- added link r_arm_pitch, mass 0.962; visual mesh filename=../../meshes/r_arm_pitch.STL
- added link r_arm_roll, mass 0.57; visual mesh filename=../../meshes/r_arm_roll.STL
- added link r_arm_yaw, mass 1.65; visual mesh filename=../../meshes/r_arm_yaw.STL
- added link r_forearm_pitch, mass 0.429; visual mesh filename=../../meshes/r_foream.STL
- added link r_hand_pitch, mass 0.331; visual mesh filename=../../meshes/r_hand_roll.STL
- added link r_hand_roll, mass 0.64; visual mesh filename=../../meshes/r_hand_pitch.STL
- added link r_hand_yaw, mass 0.61; visual mesh filename=../../meshes/r_hand_yaw.STL
Joints:
- removed joint zarm_l1_joint
- removed joint zarm_l2_joint
- removed joint zarm_l3_joint
- removed joint zarm_l4_joint
- removed joint zarm_l5_joint
- removed joint zarm_l6_joint
- removed joint zarm_l7_joint
- removed joint zarm_r1_joint
- removed joint zarm_r2_joint
- removed joint zarm_r3_joint
- removed joint zarm_r4_joint
- removed joint zarm_r5_joint
- removed joint zarm_r6_joint
- removed joint zarm_r7_joint
- added joint l_arm_pitch: type continuous, parent torso, child l_arm_pitch, origin xyz=-0.0174998525199963 0.2927 0.324500000000001 rpy=0 0 0, axis 0 1 0, limit lower=-2.0933 upper=1.5233 effort=100 velocity=100
- added joint l_arm_roll: type continuous, parent l_arm_pitch, child l_arm_roll, origin xyz=0 0 0 rpy=0 0 0, axis 1 0 0, limit lower=-1.57 upper=2.0933 effort=100 velocity=100
- added joint l_arm_yaw: type continuous, parent l_arm_roll, child l_arm_yaw, origin xyz=0 0 0 rpy=0 0 0, axis 0 0 1, limit lower=-1.57 upper=1.57 effort=100 velocity=100
- added joint l_forearm_pitch: type continuous, parent l_arm_yaw, child l_forearm_pitch, origin xyz=0.0200000000000006 0 -0.2837 rpy=0 0 0, axis 0 1 0, limit lower=-2.44 upper=1.57 effort=100 velocity=100
- added joint l_hand_pitch: type continuous, parent l_hand_yaw, child l_hand_pitch, origin xyz=0.000199999999999024 0 -0.106462725738415 rpy=0 0 0, axis 1 0 0, limit lower=-1.57 upper=1.57 effort=100 velocity=100
- added joint l_hand_roll: type continuous, parent l_hand_pitch, child l_hand_roll, origin xyz=0 0 -0.0209999999999996 rpy=0 0 0, axis 0 1 0, limit lower=-1.657 upper=1.657 effort=100 velocity=100
- added joint l_hand_yaw: type continuous, parent l_forearm_pitch, child l_hand_yaw, origin xyz=-0.0200000000000011 0 -0.127037274261586 rpy=0 0 0, axis 0 0 1, limit lower=-1.657 upper=1.657 effort=100 velocity=100
- added joint r_arm_pitch: type continuous, parent torso, child r_arm_pitch, origin xyz=-0.0174998525199963 -0.2927 0.324500000000001 rpy=0 0 0, axis 0 1 0, limit lower=-2.0933 upper=1.5233 effort=100 velocity=100
- added joint r_arm_roll: type continuous, parent r_arm_pitch, child r_arm_roll, origin xyz=0 0 0 rpy=0 0 0, axis 1 0 0, limit lower=-1.57 upper=2.0933 effort=100 velocity=100
- added joint r_arm_yaw: type continuous, parent r_arm_roll, child r_arm_yaw, origin xyz=0 0 0 rpy=0 0 0, axis 0 0 1, limit lower=-1.57 upper=1.57 effort=100 velocity=100
- added joint r_forearm_pitch: type continuous, parent r_arm_yaw, child r_forearm_pitch, origin xyz=0.0200000000000024 0 -0.2837 rpy=0 0 0, axis 0 1 0, limit lower=-2.44 upper=1.57 effort=100 velocity=100
- added joint r_hand_pitch: type continuous, parent r_hand_yaw, child r_hand_pitch, origin xyz=0 0 -0.106462725738415 rpy=0 0 0, axis 1 0 0, limit lower=-1.57 upper=1.57 effort=100 velocity=100
- added joint r_hand_roll: type continuous, parent r_hand_pitch, child r_hand_roll, origin xyz=0 0 -0.0209999999999999 rpy=0 0 0, axis 0 1 0, limit lower=-1.657 upper=1.657 effort=100 velocity=100
- added joint r_hand_yaw: type continuous, parent r_forearm_pitch, child r_hand_yaw, origin xyz=-0.0200000000000001 0 -0.127037274261587 rpy=0 0 0, axis 0 0 1, limit lower=-1.657 upper=1.657 effort=100 velocity=100
- joint zarm_l7_end_effector_joint: parent zarm_l7_link -> l_hand_roll
- joint zarm_r7_end_effector_joint: parent zarm_r7_link -> r_hand_roll

Commit message: sync https://www.lejuhub.com/highlydynamic/kuavo-ros-control/commit/be7a871fd7b071fc0fa3ce3bec0d5d8ec5e98a4b

File: src/kuavo_assets/models/biped_s43/urdf/drake/biped_v3_arm.urdf (robot description, URDF)
Before this commit: robot biped_v3_arm, 17 links, 16 joints
Links:
- removed link l_arm_pitch
- removed link l_arm_roll
- removed link l_arm_yaw
- removed link l_forearm_pitch
- removed link l_hand_pitch
- removed link l_hand_roll
- removed link l_hand_yaw
- removed link r_arm_pitch
- removed link r_arm_roll
- removed link r_arm_yaw
- removed link r_forearm_pitch
- removed link r_hand_pitch
- removed link r_hand_roll
- removed link r_hand_yaw
- added link zarm_l1_link, mass 0.962; visual mesh filename=../../meshes/l_arm_pitch.STL
- added link zarm_l2_link, mass 0.57; visual mesh filename=../../meshes/l_arm_roll.STL
- added link zarm_l3_link, mass 1.65; visual mesh filename=../../meshes/l_arm_yaw.STL
- added link zarm_l4_link, mass 0.429; visual mesh filename=../../meshes/l_foream.STL
- added link zarm_l5_link, mass 0.61; visual mesh filename=../../meshes/l_hand_yaw.STL
- added link zarm_l6_link, mass 0.331; visual mesh filename=../../meshes/l_hand_roll.STL
- added link zarm_l7_link, mass 0.64; visual mesh filename=../../meshes/l_hand_pitch.STL
- added link zarm_r1_link, mass 0.962; visual mesh filename=../../meshes/r_arm_pitch.STL
- added link zarm_r2_link, mass 0.57; visual mesh filename=../../meshes/r_arm_roll.STL
- added link zarm_r3_link, mass 1.65; visual mesh filename=../../meshes/r_arm_yaw.STL
- added link zarm_r4_link, mass 0.429; visual mesh filename=../../meshes/r_foream.STL
- added link zarm_r5_link, mass 0.61; visual mesh filename=../../meshes/r_hand_yaw.STL
- added link zarm_r6_link, mass 0.331; visual mesh filename=../../meshes/r_hand_roll.STL
- added link zarm_r7_link, mass 0.64; visual mesh filename=../../meshes/r_hand_pitch.STL
Joints:
- removed joint l_arm_pitch
- removed joint l_arm_roll
- removed joint l_arm_yaw
- removed joint l_forearm_pitch
- removed joint l_hand_pitch
- removed joint l_hand_roll
- removed joint l_hand_yaw
- removed joint r_arm_pitch
- removed joint r_arm_roll
- removed joint r_arm_yaw
- removed joint r_forearm_pitch
- removed joint r_hand_pitch
- removed joint r_hand_roll
- removed joint r_hand_yaw
- added joint zarm_l1_joint: type continuous, parent torso, child zarm_l1_link, origin xyz=-0.0174998525199963 0.2927 0.324500000000001 rpy=0 0 0, axis 0 1 0, limit lower=-2.0933 upper=1.5233 effort=100 velocity=100
- added joint zarm_l2_joint: type continuous, parent zarm_l1_link, child zarm_l2_link, origin xyz=0 0 0 rpy=0 0 0, axis 1 0 0, limit lower=-1.57 upper=2.0933 effort=100 velocity=100
- added joint zarm_l3_joint: type continuous, parent zarm_l2_link, child zarm_l3_link, origin xyz=0 0 0 rpy=0 0 0, axis 0 0 1, limit lower=-1.57 upper=1.57 effort=100 velocity=100
- added joint zarm_l4_joint: type continuous, parent zarm_l3_link, child zarm_l4_link, origin xyz=0.0200000000000006 0 -0.2837 rpy=0 0 0, axis 0 1 0, limit lower=-2.44 upper=1.57 effort=100 velocity=100
- added joint zarm_l5_joint: type continuous, parent zarm_l4_link, child zarm_l5_link, origin xyz=-0.0200000000000011 0 -0.127037274261586 rpy=0 0 0, axis 0 0 1, limit lower=-1.657 upper=1.657 effort=100 velocity=100
- added joint zarm_l6_joint: type continuous, parent zarm_l5_link, child zarm_l6_link, origin xyz=0.000199999999999024 0 -0.106462725738415 rpy=0 0 0, axis 1 0 0, limit lower=-1.57 upper=1.57 effort=100 velocity=100
- added joint zarm_l7_joint: type continuous, parent zarm_l6_link, child zarm_l7_link, origin xyz=0 0 -0.0209999999999996 rpy=0 0 0, axis 0 1 0, limit lower=-1.657 upper=1.657 effort=100 velocity=100
- added joint zarm_r1_joint: type continuous, parent torso, child zarm_r1_link, origin xyz=-0.0174998525199963 -0.2927 0.324500000000001 rpy=0 0 0, axis 0 1 0, limit lower=-2.0933 upper=1.5233 effort=100 velocity=100
- added joint zarm_r2_joint: type continuous, parent zarm_r1_link, child zarm_r2_link, origin xyz=0 0 0 rpy=0 0 0, axis 1 0 0, limit lower=-1.57 upper=2.0933 effort=100 velocity=100
- added joint zarm_r3_joint: type continuous, parent zarm_r2_link, child zarm_r3_link, origin xyz=0 0 0 rpy=0 0 0, axis 0 0 1, limit lower=-1.57 upper=1.57 effort=100 velocity=100
- added joint zarm_r4_joint: type continuous, parent zarm_r3_link, child zarm_r4_link, origin xyz=0.0200000000000024 0 -0.2837 rpy=0 0 0, axis 0 1 0, limit lower=-2.44 upper=1.57 effort=100 velocity=100
- added joint zarm_r5_joint: type continuous, parent zarm_r4_link, child zarm_r5_link, origin xyz=-0.0200000000000001 0 -0.127037274261587 rpy=0 0 0, axis 0 0 1, limit lower=-1.657 upper=1.657 effort=100 velocity=100
- added joint zarm_r6_joint: type continuous, parent zarm_r5_link, child zarm_r6_link, origin xyz=0 0 -0.106462725738415 rpy=0 0 0, axis 1 0 0, limit lower=-1.57 upper=1.57 effort=100 velocity=100
- added joint zarm_r7_joint: type continuous, parent zarm_r6_link, child zarm_r7_link, origin xyz=0 0 -0.0209999999999999 rpy=0 0 0, axis 0 1 0, limit lower=-1.657 upper=1.657 effort=100 velocity=100
- joint zarm_l7_end_effector_joint: parent l_hand_roll -> zarm_l7_link
- joint zarm_r7_end_effector_joint: parent r_hand_roll -> zarm_r7_link

Commit message: sync https://www.lejuhub.com/highlydynamic/kuavo-ros-control/commit/68ccc3d6ea8775a51bbb106c6fbf7531ad5f93ca

File: src/kuavo_assets/models/biped_s43/urdf/drake/biped_v3_arm.urdf (robot description, URDF)
Before this commit: robot biped_v3_arm, 17 links, 16 joints
Joints:
- joint zarm_l1_joint: limit lower=-2.0933 upper=1.5233 effort=100 velocity=100 -> lower=-3.1415 upper=1.57 effort=100 velocity=100; type continuous -> revolute
- joint zarm_l2_joint: limit lower=-1.57 upper=2.0933 effort=100 velocity=100 -> lower=-0.348 upper=2.0933 effort=100 velocity=100; type continuous -> revolute
- joint zarm_l3_joint: type continuous -> revolute
- joint zarm_l4_joint: limit lower=-2.44 upper=1.57 effort=100 velocity=100 -> lower=-2.616 upper=0 effort=100 velocity=100; type continuous -> revolute
- joint zarm_l5_joint: limit lower=-1.657 upper=1.657 effort=100 velocity=100 -> lower=-1.57 upper=1.57 effort=100 velocity=100; type continuous -> revolute
- joint zarm_l6_joint: limit lower=-1.57 upper=1.57 effort=100 velocity=100 -> lower=-0.697 upper=0.697 effort=100 velocity=100; type continuous -> revolute
- joint zarm_l7_joint: limit lower=-1.657 upper=1.657 effort=100 velocity=100 -> lower=-1.3083 upper=0.697 effort=100 velocity=100; type continuous -> revolute
- joint zarm_r1_joint: limit lower=-2.0933 upper=1.5233 effort=100 velocity=100 -> lower=-3.1415 upper=1.57 effort=100 velocity=100; type continuous -> revolute
- joint zarm_r2_joint: limit lower=-1.57 upper=2.0933 effort=100 velocity=100 -> lower=-2.0933 upper=0.3488 effort=100 velocity=100; type continuous -> revolute
- joint zarm_r3_joint: type continuous -> revolute
- joint zarm_r4_joint: limit lower=-2.44 upper=1.57 effort=100 velocity=100 -> lower=-2.61 upper=0 effort=100 velocity=100; type continuous -> revolute
- joint zarm_r5_joint: limit lower=-1.657 upper=1.657 effort=100 velocity=100 -> lower=-1.57 upper=1.57 effort=100 velocity=100; type continuous -> revolute
- joint zarm_r6_joint: limit lower=-1.57 upper=1.57 effort=100 velocity=100 -> lower=-0.697 upper=0.697 effort=100 velocity=100; type continuous -> revolute
- joint zarm_r7_joint: limit lower=-1.657 upper=1.657 effort=100 velocity=100 -> lower=-0.6977 upper=1.3083 effort=100 velocity=100; type continuous -> revolute
