Commit message: sync https://www.lejuhub.com/highlydynamic/kuavo-ros-control/commit/d0fe790568d694d8704ed60cf13705df52faa392

File: src/kuavo_assets/models/biped_s42/urdf/biped_s42.urdf (robot description, URDF)
Before this commit: robot biped_s42, 45 links, 44 joints
Links:
- link base_link: mass 25.1666 -> 26.5696

File: src/kuavo_assets/models/biped_s42/urdf/drake/biped_v3.urdf (robot description, URDF)
Before this commit: robot biped_v3, 13 links, 12 joints
Links:
- link torso: mass 33.83884316 -> 35.24184316

File: src/kuavo_assets/models/biped_s42/urdf/drake/biped_v3_all_joint.urdf (robot description, URDF)
Before this commit: robot biped_v3_all_joint, 35 links, 30 joints
Links:
- link torso: mass 25.23624316 -> 26.63924316

File: src/kuavo_assets/models/biped_s42/urdf/drake/biped_v3_full.urdf (robot description, URDF)
Before this commit: robot biped_v3_full, 27 links, 26 joints
Links:
- link torso: mass 25.87904316 -> 27.28204316

File: src/kuavo_assets/models/biped_s43/urdf/biped_s43.urdf (robot description, URDF)
Before this commit: robot biped_s4, 45 links, 44 joints
Joints:
- joint zarm_r2_joint: limit lower=0.3489 upper=-2.0933 effort=8.5 velocity=9 -> lower=-0.3489 upper=2.0933 effort=8.5 velocity=9

File: src/kuavo_assets/models/biped_s43/urdf/drake/biped_v3_arm.urdf (robot description, URDF)
Before this commit: robot biped_v3_arm, 17 links, 16 joints
Joints:
- joint zarm_l1_joint: limit lower=-3.1415 upper=1.57 effort=100 velocity=100 -> lower=-2.0933 upper=1.5233 effort=100 velocity=100; type revolute -> continuous
- joint zarm_l2_joint: limit lower=-0.348 upper=2.0933 effort=100 velocity=100 -> lower=-1.57 upper=2.0933 effort=100 velocity=100; type revolute -> continuous
- joint zarm_l3_joint: type revolute -> continuous
- joint zarm_l4_joint: limit lower=-2.616 upper=0 effort=100 velocity=100 -> lower=-2.44 upper=1.57 effort=100 velocity=100; type revolute -> continuous
- joint zarm_l5_joint: limit lower=-1.57 upper=1.57 effort=100 velocity=100 -> lower=-1.657 upper=1.657 effort=100 velocity=100; type revolute -> continuous
- joint zarm_l6_joint: limit lower=-0.697 upper=0.697 effort=100 velocity=100 -> lower=-1.57 upper=1.57 effort=100 velocity=100; type revolute -> continuous
- joint zarm_l7_joint: limit lower=-1.3083 upper=0.697 effort=100 velocity=100 -> lower=-1.657 upper=1.657 effort=100 velocity=100; type revolute -> continuous
- joint zarm_r1_joint: limit lower=-3.1415 upper=1.57 effort=100 velocity=100 -> lower=-2.0933 upper=1.5233 effort=100 velocity=100; type revolute -> continuous
- joint zarm_r2_joint: limit lower=-2.0933 upper=0.3488 effort=100 velocity=100 -> lower=-1.57 upper=2.0933 effort=100 velocity=100; type revolute -> continuous
- joint zarm_r3_joint: type revolute -> continuous
- joint zarm_r4_joint: limit lower=-2.61 upper=0 effort=100 velocity=100 -> lower=-2.44 upper=1.57 effort=100 velocity=100; type revolute -> continuous
- joint zarm_r5_joint: limit lower=-1.57 upper=1.57 effort=100 velocity=100 -> lower=-1.657 upper=1.657 effort=100 velocity=100; type revolute -> continuous
- joint zarm_r6_joint: limit lower=-0.697 upper=0.697 effort=100 velocity=100 -> lower=-1.57 upper=1.57 effort=100 velocity=100; type revolute -> continuous
- joint zarm_r7_joint: limit lower=-0.6977 upper=1.3083 effort=100 velocity=100 -> lower=-1.657 upper=1.657 effort=100 velocity=100; type revolute -> continuous

Commit message: init

File: src/kuavo_assets/models/biped_s42/urdf/biped_s42.urdf (robot description, URDF)
Before this commit: robot biped_s42, 45 links, 44 joints
Links:
- link base_link: mass 26.5696 -> 25.2696

File: src/kuavo_assets/models/biped_s42/urdf/drake/biped_v3.urdf (robot description, URDF)
Before this commit: robot biped_v3, 13 links, 12 joints
Links:
- link torso: mass 35.24184316 -> 33.94184316

File: src/kuavo_assets/models/biped_s42/urdf/drake/biped_v3_all_joint.urdf (robot description, URDF)
Before this commit: robot biped_v3_all_joint, 35 links, 30 joints
Links:
- link torso: mass 26.63924316 -> 25.33924316

File: src/kuavo_assets/models/biped_s42/urdf/drake/biped_v3_full.urdf (robot description, URDF)
Before this commit: robot biped_v3_full, 27 links, 26 joints
Links:
- link torso: mass 27.28204316 -> 25.98204316
